File: ctrl.kicad_pcb (KiCad board)
At the start: 2 copper layers, 100.3 x 43.2 mm, 56 parts, among them J1 OSC-I, J10 LCDD/DAH, J11 ROT/S, J12 GND, J13 BAND/SIDE, J14 GND, J15 TX/KEY, J16 OSC-TX, J17 Supply, J18 PTT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

Commit message: Fixed minors.
Connections:
- J10 pad 5: Dah -> LCD_EN
- J4 pad 5: SDA -> LCD_RS
- J5 pad 2: SDA -> LCD_RS
- J9 pad 1: LCD_RS -> Dit
- J9 pad 2: LCD_EN -> Dah
- U2 pad 11: LCD_RS -> Dit
- U2 pad 12: LCD_EN -> Dah
- U2 pad 27: SDA -> LCD_RS
- U2 pad 6: Dah -> LCD_EN
Routing:
- net SDA: track 32.6 -> 0.00 mm
- net LCD_RS: track 5.08 -> 32.6 mm
- net Dit: track 0.00 -> 5.08 mm
Other:
- board text added: "D4 D5 D6 D7 EN"
- board text added: "DIT DAH"
- board text removed: "D4 D5 D6 D7 Dah"
- board text removed: "DIT EN"
