File: trx.sch (KiCad schematic (older format))
At the start: 99 parts, among them J1 12V, J2 HF, J3 Volume, J4 Conn_01x04, J5 HP, J6 OSC-I, J7 OSC-Q, J8 TX, J9 12V, Q1 BS170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

Commit message: Backup.
Parts:
- U1, U2, U3, U6, U7: value TL072 -> LM833
- U5: value TL072 -> TLC272
Changed lines of the file:
@@
 P 1200 7000
 F 0 "U1" H 1158 7046 50  0000 L CNN
-F 1 "TL072" H 1158 6955 50  0000 L CNN
+F 1 "LM833" H 1158 6955 50  0000 L CNN
 F 2 "Package_DIP:DIP-8_W7.62mm_LongPads" H 1200 7000 50  0001 C CNN
 F 3 "http://www.ti.com/lit/ds/symlink/tl071.pdf" H 1200 7000 50  0001 C CNN
@@
 P 1800 7000
 F 0 "U2" H 1758 7046 50  0000 L CNN
-F 1 "TL072" H 1758 6955 50  0000 L CNN
+F 1 "LM833" H 1758 6955 50  0000 L CNN
 F 2 "Package_DIP:DIP-8_W7.62mm_LongPads" H 1800 7000 50  0001 C CNN
 F 3 "http://www.ti.com/lit/ds/symlink/tl071.pdf" H 1800 7000 50  0001 C CNN
@@
 P 2400 7000
 F 0 "U3" H 2358 7046 50  0000 L CNN
-F 1 "TL072" H 2358 6955 50  0000 L CNN
+F 1 "LM833" H 2358 6955 50  0000 L CNN
 F 2 "Package_DIP:DIP-8_W7.62mm_LongPads" H 2400 7000 50  0001 C CNN
 F 3 "http://www.ti.com/lit/ds/symlink/tl071.pdf" H 2400 7000 50  0001 C CNN
@@
 P 3000 7000
 F 0 "U5" H 2958 7046 50  0000 L CNN
-F 1 "TL072" H 2958 6955 50  0000 L CNN
+F 1 "TLC272" H 2958 6955 50  0000 L CNN
 F 2 "Package_DIP:DIP-8_W7.62mm_LongPads" H 3000 7000 50  0001 C CNN
 F 3 "http://www.ti.com/lit/ds/symlink/tl071.pdf" H 3000 7000 50  0001 C CNN
@@
 P 3600 7000
 F 0 "U6" H 3558 7046 50  0000 L CNN
-F 1 "TL072" H 3558 6955 50  0000 L CNN
+F 1 "LM833" H 3558 6955 50  0000 L CNN
 F 2 "Package_DIP:DIP-8_W7.62mm_LongPads" H 3600 7000 50  0001 C CNN
 F 3 "http://www.ti.com/lit/ds/symlink/tl071.pdf" H 3600 7000 50  0001 C CNN
@@
 P 4200 7000
 F 0 "U7" H 4158 7046 50  0000 L CNN
-F 1 "TL072" H 4158 6955 50  0000 L CNN
+F 1 "LM833" H 4158 6955 50  0000 L CNN
 F 2 "Package_DIP:DIP-8_W7.62mm_LongPads" H 4200 7000 50  0001 C CNN
 F 3 "http://www.ti.com/lit/ds/symlink/tl071.pdf" H 4200 7000 50  0001 C CNN

Commit message: Fixed minors.
Parts:
- R9: value 33k -> 3,3k
Changed lines of the file:
@@
 P 3050 5500
 F 0 "R9" V 2843 5500 50  0000 C CNN
-F 1 "33k" V 2934 5500 50  0000 C CNN
+F 1 "3,3k" V 2934 5500 50  0000 C CNN
 F 2 "Resistor_THT:R_Axial_DIN0204_L3.6mm_D1.6mm_P7.62mm_Horizontal" V 2980 5500 50  0001 C CNN
 F 3 "~" H 3050 5500 50  0001 C CNN

Commit message: Added libs and fixed footprints.
Parts:
- T1: footprint Transformer_THT:Transformer_Toroid_Tapped_Vertical_D10.5mm_Amidon-T37 -> DM3MAT:Transformer_1P_2S_Toroid_Vertical_D10.5mm_Amidon-T37_Wide
Changed lines of the file:
@@
 EESchema Schematic File Version 4
 LIBS:trx-cache
-EELAYER 26 0
+EELAYER 30 0
 EELAYER END
 $Descr A4 11693 8268
@@
 F 0 "T1" H 1550 2578 50  0000 C CNN
 F 1 "10:10:10 @ FT37-43" H 1550 2487 50  0000 C CNN
-F 2 "Transformer_THT:Transformer_Toroid_Tapped_Vertical_D10.5mm_Amidon-T37" H 1550 2000 50  0001 C CNN
+F 2 "DM3MAT:Transformer_1P_2S_Toroid_Vertical_D10.5mm_Amidon-T37_Wide" H 1550 2000 50  0001 C CNN
 F 3 "~" H 1550 2000 50  0001 C CNN
 	1    1550 2000
