File: pa.kicad_pcb (KiCad board)
At the start: 2 copper layers, 100.3 x 71.1 mm, 91 parts, among them J1 Conn_Coaxial, J10 TX5V, J11 12V-PA, J12 12V, J2 20m, J3 40m, J4 80m, J5 Key5V, J6 RX-HF, J7 TX-HF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

Commit message: backup.
Parts:
- C12, C17, C4, C7: value 680p -> 330p
- C13, C8: value 1n -> 680p
- C14, C9: value 1.8n -> 1n
- C15, C2: value 120p -> 100p
- C16, C3: value 470p -> 150p
- C18, C5: value 1n -> 470p
- L1, L9: value 363n -> 440n
- L10, L2: value 610n -> 650n
- L11, L3: value 1460n -> 1330n
- L12, L4: value 2520n -> 2050n
- L5: value 432n -> 520n
- L6: value 640n -> 760n
- L7: value 1570n -> 1530n
- L8: value 2780n -> 3000n
- T1: value 10:10@FT37-43 -> 8+8@FT37-43; footprint Transformer_THT:Transformer_Toroid_Vertical_D10.5mm_Amidon-T37 -> DM3MAT:Transformer_1P_1S_Toroid_Vertical_D10.5mm_Amidon-T37
- moved T1 4.02 mm to (127.0, 113.0), turned to 90 degrees
Routing:
- net Net-(Q11-Pad1): vias 0 -> 2
- net GND: vias 189 -> 187

Commit message: Added libs and fixed footprints.
Connections:
- K1 pad 12: (no net) -> Net-(K1-Pad12)
- K1 pad 22: (no net) -> Net-(K1-Pad22)
- K2 pad 12: (no net) -> Net-(K2-Pad12)
- K2 pad 22: (no net) -> Net-(K2-Pad22)
- K3 pad 12: (no net) -> Net-(K3-Pad12)
- K3 pad 22: (no net) -> Net-(K3-Pad22)
- K4 pad 12: (no net) -> Net-(K4-Pad12)
- K4 pad 22: (no net) -> Net-(K4-Pad22)
Routing:
- net Net-(Q11-Pad1): vias 2 -> 0
- net GND: vias 187 -> 189

Commit message: Updated library.
Parts:
- moved T1 2.54 mm to (129.5, 113.0)
Changed lines of the file:
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@@
       (effects (font (size 1 1) (thickness 0.15)))
     )
-    (fp_text user A (at 4.66 0 180) (layer F.Fab)
+    (fp_text user A (at 4.66 0) (layer F.Fab)
       (effects (font (size 1 1) (thickness 0.15)))
     )
@@
       (effects (font (size 1 1) (thickness 0.15)))
     )
-    (fp_text user K (at -1.905 0 180) (layer F.SilkS)
+    (fp_text user K (at 0 -2) (layer F.Fab)
       (effects (font (size 1 1) (thickness 0.15)))
     )
@@
       (effects (font (size 1 1) (thickness 0.15)))
     )
-    (fp_text user K (at 0 -2 180) (layer F.Fab)
+    (fp_text user K (at 0 -2) (layer F.Fab)
       (effects (font (size 1 1) (thickness 0.15)))
     )
@@
       (effects (font (size 1 1) (thickness 0.15)))
     )
-    (fp_text user K (at 0 -2 180) (layer F.Fab)
+    (fp_text user K (at 0 -2) (layer F.Fab)
       (effects (font (size 1 1) (thickness 0.15)))
     )
@@
       (effects (font (size 1 1) (thickness 0.15)))
     )
-    (fp_text user K (at -1.905 0 180) (layer F.SilkS)
+    (fp_text user K (at 0 -2) (layer F.Fab)
       (effects (font (size 1 1) (thickness 0.15)))
     )
@@
   )
   (module DM3MAT:Transformer_1P_1S_Toroid_Vertical_D10.5mm_Amidon-T37 (layer F.Cu)
-    (at 127 113.03 90)
+    (at 129.54 113.03 90)
     (descr "L_Toroid, Vertical series, Radial, pin pitch=5.08mm, , length*width=10*5mm^2")
     (tags "L_Toroid Vertical series Radial pin pitch 5.08mm  length 10mm width 5mm")
@@
       (effects (font (size 1 1) (thickness 0.15)))
     )
-    (fp_line (start 6.35 -1.25) (end -6.35 -1.25) (layer F.CrtYd) (width 0.05))
-    (fp_line (start 6.35 6.33) (end 6.35 -1.25) (layer F.CrtYd) (width 0.05))
-    (fp_line (start -6.35 6.33) (end 6.35 6.33) (layer F.CrtYd) (width 0.05))
-    (fp_line (start -6.35 -1.25) (end -6.35 6.33) (layer F.CrtYd) (width 0.05))
-    (fp_line (start 5.12 -0.08) (end 5.12 3.81) (layer F.SilkS) (width 0.12))
-    (fp_line (start -5.12 1.27) (end -5.12 5.16) (layer F.SilkS) (width 0.12))
-    (fp_line (start -5.12 5.16) (end 1.27 5.16) (layer F.SilkS) (width 0.12))
-    (fp_line (start -1.27 -0.08) (end 5.12 -0.08) (layer F.SilkS) (width 0.12))
-    (fp_line (start 3.2 0) (end 3.6 5.08) (layer F.Fab) (width 0.1))
-    (fp_line (start 2.4 0) (end 2.8 5.08) (layer F.Fab) (width 0.1))
-    (fp_line (start 1.6 0) (end 2 5.08) (layer F.Fab) (width 0.1))
-    (fp_line (start 0.8 0) (end 1.2 5.08) (layer F.Fab) (width 0.1))
-    (fp_line (start 0 0) (end 0.4 5.08) (layer F.Fab) (width 0.1))
-    (fp_line (start -0.8 0) (end -0.4 5.08) (layer F.Fab) (width 0.1))
-    (fp_line (start -1.6 0) (end -1.2 5.08) (layer F.Fab) (width 0.1))
-    (fp_line (start -2.4 0) (end -2 5.08) (layer F.Fab) (width 0.1))
-    (fp_line (start -3.2 0) (end -2.8 5.08) (layer F.Fab) (width 0.1))
-    (fp_line (start -4 0) (end -3.6 5.08) (layer F.Fab) (width 0.1))
-    (fp_line (start 4 0) (end -4 0) (layer F.Fab) (width 0.1))
-    (fp_line (start 4 5.08) (end 4 0) (layer F.Fab) (width 0.1))
-    (fp_line (start -4 5.08) (end 4 5.08) (layer F.Fab) (width 0.1))
-    (fp_line (start -4 0) (end -4 5.08) (layer F.Fab) (width 0.1))
-    (fp_line (start 5 0.04) (end -5 0.04) (layer F.Fab) (width 0.1))
-    (fp_line (start 5 5.04) (end 5 0.04) (layer F.Fab) (width 0.1))
-    (fp_line (start -5 5.04) (end 5 5.04) (layer F.Fab) (width 0.1))
-    (fp_line (start -5 0.04) (end -5 5.04) (layer F.Fab) (width 0.1))
-    (pad 4 thru_hole circle (at -2.54 0 90) (size 2 2) (drill 1) (layers *.Cu *.Mask)
+    (fp_line (start 6.35 -3.79) (end -6.35 -3.79) (layer F.CrtYd) (width 0.05))
+    (fp_line (start 6.35 3.79) (end 6.35 -3.79) (layer F.CrtYd) (width 0.05))
+    (fp_line (start -6.35 3.79) (end 6.35 3.79) (layer F.CrtYd) (width 0.05))
+    (fp_line (start -6.35 -3.79) (end -6.35 3.79) (layer F.CrtYd) (width 0.05))
+    (fp_line (start 5.12 -2.62) (end 5.12 1.27) (layer F.SilkS) (width 0.12))
+    (fp_line (start -5.12 -1.27) (end -5.12 2.62) (layer F.SilkS) (width 0.12))
+    (fp_line (start -5.12 2.62) (end 1.27 2.62) (layer F.SilkS) (width 0.12))
+    (fp_line (start -1.27 -2.62) (end 5.12 -2.62) (layer F.SilkS) (width 0.12))
+    (fp_line (start 3.2 -2.54) (end 3.6 2.54) (layer F.Fab) (width 0.1))
+    (fp_line (start 2.4 -2.54) (end 2.8 2.54) (layer F.Fab) (width 0.1))
+    (fp_line (start 1.6 -2.54) (end 2 2.54) (layer F.Fab) (width 0.1))
+    (fp_line (start 0.8 -2.54) (end 1.2 2.54) (layer F.Fab) (width 0.1))
+    (fp_line (start 0 -2.54) (end 0.4 2.54) (layer F.Fab) (width 0.1))
+    (fp_line (start -0.8 -2.54) (end -0.4 2.54) (layer F.Fab) (width 0.1))
+    (fp_line (start -1.6 -2.54) (end -1.2 2.54) (layer F.Fab) (width 0.1))
+    (fp_line (start -2.4 -2.54) (end -2 2.54) (layer F.Fab) (width 0.1))
+    (fp_line (start -3.2 -2.54) (end -2.8 2.54) (layer F.Fab) (width 0.1))
+    (fp_line (start -4 -2.54) (end -3.6 2.54) (layer F.Fab) (width 0.1))
+    (fp_line (start 4 -2.54) (end -4 -2.54) (layer F.Fab) (width 0.1))
+    (fp_line (start 4 2.54) (end 4 -2.54) (layer F.Fab) (width 0.1))
+    (fp_line (start -4 2.54) (end 4 2.54) (layer F.Fab) (width 0.1))
+    (fp_line (start -4 -2.54) (end -4 2.54) (layer F.Fab) (width 0.1))
+    (fp_line (start 5 -2.5) (end -5 -2.5) (layer F.Fab) (width 0.1))
+    (fp_line (start 5 2.5) (end 5 -2.5) (layer F.Fab) (width 0.1))
+    (fp_line (start -5 2.5) (end 5 2.5) (layer F.Fab) (width 0.1))
+    (fp_line (start -5 -2.5) (end -5 2.5) (layer F.Fab) (width 0.1))
+    (pad 4 thru_hole circle (at -2.54 -2.54 90) (size 2 2) (drill 1) (layers *.Cu *.Mask)
       (net 22 "Net-(C23-Pad2)"))
-    (pad 1 thru_hole circle (at -5.08 0 90) (size 2 2) (drill 1) (layers *.Cu *.Mask)
+    (pad 1 thru_hole circle (at -5.08 -2.54 90) (size 2 2) (drill 1) (layers *.Cu *.Mask)
       (net 48 "Net-(Q11-Pad1)"))
-    (pad 2 thru_hole circle (at 2.54 5.08 90) (size 2 2) (drill 1) (layers *.Cu *.Mask)
+    (pad 2 thru_hole circle (at 2.54 2.54 90) (size 2 2) (drill 1) (layers *.Cu *.Mask)
       (net 20 "Net-(C20-Pad2)"))
-    (pad 3 thru_hole circle (at 5.08 5.08 90) (size 2 2) (drill 1) (layers *.Cu *.Mask)
+    (pad 3 thru_hole circle (at 5.08 2.54 90) (size 2 2) (drill 1) (layers *.Cu *.Mask)
       (net 48 "Net-(Q11-Pad1)"))
     (model ${KISYS3DMOD}/Inductor_THT.3dshapes/L_Toroid_Vertical_L10.0mm_W5.0mm_P5.08mm.wrl
@@
       (rotate (xyz 0 0 0))
     )
+    (model /home/hannes/AFU/kicad/DM3MAT/DM3MAT.3dshapes/Transformer_1P_1S_Toroid_Vertical_D10.5mm_Amidon-T37.step
+      (at (xyz 0 0 0))
+      (scale (xyz 1 1 1))
+      (rotate (xyz 0 0 0))
+    )
   )
   (module Connector_Coaxial:BNC_horizontal (layer F.Cu)
@@
   (segment (start 132.08 113.03) (end 134.62 113.03) (width 0.5) (layer B.Cu) (net 2))
   (via (at 132.08 113.03) (size 0.8) (drill 0.4) (layers F.Cu B.Cu) (net 2))
-  (via (at 129.54 107.95) (size 0.8) (drill 0.4) (layers F.Cu B.Cu) (net 2))
   (via (at 129.54 118.11) (size 0.8) (drill 0.4) (layers F.Cu B.Cu) (net 2))
   (via (at 151.13 97.79) (size 0.8) (drill 0.4) (layers F.Cu B.Cu) (net 2))
@@
   (via (at 193.04 88.9) (size 0.8) (drill 0.4) (layers F.Cu B.Cu) (net 2))
   (via (at 190.5 87.63) (size 0.8) (drill 0.4) (layers F.Cu B.Cu) (net 2))
+  (via (at 132.08 115.57) (size 0.8) (drill 0.4) (layers F.Cu B.Cu) (net 2))
+  (via (at 132.08 118.11) (size 0.8) (drill 0.4) (layers F.Cu B.Cu) (net 2))
+  (via (at 129.54 107.95) (size 0.8) (drill 0.4) (layers F.Cu B.Cu) (net 2))
   (segment (start 144.78 95.25) (end 144.78 100.33) (width 0.5) (layer B.Cu) (net 3) (status 30))
   (segment (start 160.02 97.75) (end 160.06 97.79) (width 0.25) (layer B.Cu) (net 4) (status 30))
@@
   (segment (start 122.08 120.65) (end 122 120.73) (width 0.5) (layer B.Cu) (net 47) (status 30))
   (segment (start 124.46 120.65) (end 122.08 120.65) (width 0.5) (layer B.Cu) (net 47) (status 30))
-  (via (at 132.08 115.57) (size 0.8) (drill 0.4) (layers F.Cu B.Cu) (net 2))
-  (via (at 132.08 118.11) (size 0.8) (drill 0.4) (layers F.Cu B.Cu) (net 2))
   (segment (start 132.08 107.95) (end 132.08 105.41) (width 0.25) (layer B.Cu) (net 48) (status 20))
   (segment (start 132.08 105.41) (end 132.08 100.33) (width 0.25) (layer B.Cu) (net 48) (status 30))
