File: pa.sch (KiCad schematic (older format))
At the start: 91 parts, among them J1 Conn_Coaxial, J10 TX5V, J11 12V-PA, J12 12V, J2 20m, J3 40m, J4 80m, J5 Key5V, J6 RX-HF, J7 TX-HF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

Commit message: Backup.
Parts:
- C12, C17, C4, C7: value 680p -> 330p
- C13, C8: value 1n -> 680p
- C14, C9: value 1.8n -> 1n
- C15, C2: value 120p -> 100p
- C16, C3: value 470p -> 150p
- C18, C5: value 1n -> 470p
- L1, L9: value 363n -> 440n
- L10, L2: value 610n -> 650n
- L11, L3: value 1460n -> 1330n
- L12, L4: value 2520n -> 2050n
- L5: value 432n -> 520n
- L6: value 640n -> 760n
- L7: value 1570n -> 1530n
- L8: value 2780n -> 3000n
Other:
- note added: "LP 60m, 40m"
- note removed: "LP 40m"
Changed lines of the file:
@@
 P 2250 3500
 F 0 "L2" V 2475 3500 50  0000 C CNN
-F 1 "610n" V 2384 3500 50  0000 C CNN
+F 1 "650n" V 2384 3500 50  0000 C CNN
 F 2 "Inductor_THT:L_Toroid_Vertical_L10.0mm_W5.0mm_P5.08mm_Diagonal" H 2250 3500 50  0001 C CNN
 F 3 "~" H 2250 3500 50  0001 C CNN
@@
 P 2000 3750
 F 0 "C3" H 2115 3796 50  0000 L CNN
-F 1 "470p" H 2115 3705 50  0000 L CNN
+F 1 "150p" H 2115 3705 50  0000 L CNN
 F 2 "Capacitor_THT:C_Disc_D3.0mm_W2.0mm_P2.50mm" H 2038 3600 50  0001 C CNN
 F 3 "~" H 2000 3750 50  0001 C CNN
@@
 P 2500 3750
 F 0 "C7" H 2615 3796 50  0000 L CNN
-F 1 "680p" H 2615 3705 50  0000 L CNN
+F 1 "330p" H 2615 3705 50  0000 L CNN
 F 2 "Capacitor_THT:C_Disc_D3.0mm_W2.0mm_P2.50mm" H 2538 3600 50  0001 C CNN
 F 3 "~" H 2500 3750 50  0001 C CNN
@@
 P 2750 3500
 F 0 "L6" V 2975 3500 50  0000 C CNN
-F 1 "640n" V 2884 3500 50  0000 C CNN
+F 1 "760n" V 2884 3500 50  0000 C CNN
 F 2 "Inductor_THT:L_Toroid_Vertical_L10.0mm_W5.0mm_P5.08mm_Diagonal" H 2750 3500 50  0001 C CNN
 F 3 "~" H 2750 3500 50  0001 C CNN
@@
 P 3000 3750
 F 0 "C12" H 3115 3796 50  0000 L CNN
-F 1 "680p" H 3115 3705 50  0000 L CNN
+F 1 "330p" H 3115 3705 50  0000 L CNN
 F 2 "Capacitor_THT:C_Disc_D3.0mm_W1.6mm_P2.50mm" H 3038 3600 50  0001 C CNN
 F 3 "~" H 3000 3750 50  0001 C CNN
@@
 P 3250 3500
 F 0 "L10" V 3475 3500 50  0000 C CNN
-F 1 "610n" V 3384 3500 50  0000 C CNN
+F 1 "650n" V 3384 3500 50  0000 C CNN
 F 2 "Inductor_THT:L_Toroid_Vertical_L10.0mm_W5.0mm_P5.08mm_Diagonal" H 3250 3500 50  0001 C CNN
 F 3 "~" H 3250 3500 50  0001 C CNN
@@
 P 3500 3750
 F 0 "C16" H 3615 3796 50  0000 L CNN
-F 1 "470p" H 3615 3705 50  0000 L CNN
+F 1 "150p" H 3615 3705 50  0000 L CNN
 F 2 "Capacitor_THT:C_Disc_D3.0mm_W2.0mm_P2.50mm" H 3538 3600 50  0001 C CNN
 F 3 "~" H 3500 3750 50  0001 C CNN
@@
 P 2250 1700
 F 0 "L1" V 2475 1700 50  0000 C CNN
-F 1 "363n" V 2384 1700 50  0000 C CNN
+F 1 "440n" V 2384 1700 50  0000 C CNN
 F 2 "Inductor_THT:L_Toroid_Vertical_L10.0mm_W5.0mm_P5.08mm_Diagonal" H 2250 1700 50  0001 C CNN
 F 3 "~" H 2250 1700 50  0001 C CNN
@@
 P 2000 1950
 F 0 "C2" H 2115 1996 50  0000 L CNN
-F 1 "120p" H 2115 1905 50  0000 L CNN
+F 1 "100p" H 2115 1905 50  0000 L CNN
 F 2 "Capacitor_THT:C_Disc_D3.0mm_W1.6mm_P2.50mm" H 2038 1800 50  0001 C CNN
 F 3 "~" H 2000 1950 50  0001 C CNN
@@
 P 2750 1700
 F 0 "L5" V 2975 1700 50  0000 C CNN
-F 1 "432n" V 2884 1700 50  0000 C CNN
+F 1 "520n" V 2884 1700 50  0000 C CNN
 F 2 "Inductor_THT:L_Toroid_Vertical_L10.0mm_W5.0mm_P5.08mm_Diagonal" H 2750 1700 50  0001 C CNN
 F 3 "~" H 2750 1700 50  0001 C CNN
@@
 P 3250 1700
 F 0 "L9" V 3475 1700 50  0000 C CNN
-F 1 "363n" V 3384 1700 50  0000 C CNN
+F 1 "440n" V 3384 1700 50  0000 C CNN
 F 2 "Inductor_THT:L_Toroid_Vertical_L10.0mm_W5.0mm_P5.08mm_Diagonal" H 3250 1700 50  0001 C CNN
 F 3 "~" H 3250 1700 50  0001 C CNN
@@
 P 3500 1950
 F 0 "C15" H 3615 1996 50  0000 L CNN
-F 1 "120p" H 3615 1905 50  0000 L CNN
+F 1 "100p" H 3615 1905 50  0000 L CNN
 F 2 "Capacitor_THT:C_Disc_D3.0mm_W2.0mm_P2.50mm" H 3538 1800 50  0001 C CNN
 F 3 "~" H 3500 1950 50  0001 C CNN
@@
 P 2250 5300
 F 0 "L3" V 2475 5300 50  0000 C CNN
-F 1 "1460n" V 2384 5300 50  0000 C CNN
+F 1 "1330n" V 2384 5300 50  0000 C CNN
 F 2 "Inductor_THT:L_Toroid_Vertical_L10.0mm_W5.0mm_P5.08mm_Diagonal" H 2250 5300 50  0001 C CNN
 F 3 "~" H 2250 5300 50  0001 C CNN
@@
 P 2000 5550
 F 0 "C4" H 2115 5596 50  0000 L CNN
-F 1 "680p" H 2115 5505 50  0000 L CNN
+F 1 "330p" H 2115 5505 50  0000 L CNN
 F 2 "Capacitor_THT:C_Disc_D3.0mm_W2.0mm_P2.50mm" H 2038 5400 50  0001 C CNN
 F 3 "~" H 2000 5550 50  0001 C CNN
@@
 P 2500 5550
 F 0 "C8" H 2615 5596 50  0000 L CNN
-F 1 "1n" H 2615 5505 50  0000 L CNN
+F 1 "680p" H 2615 5505 50  0000 L CNN
 F 2 "Capacitor_THT:C_Disc_D3.0mm_W2.0mm_P2.50mm" H 2538 5400 50  0001 C CNN
 F 3 "~" H 2500 5550 50  0001 C CNN
@@
 P 2750 5300
 F 0 "L7" V 2975 5300 50  0000 C CNN
-F 1 "1570n" V 2884 5300 50  0000 C CNN
+F 1 "1530n" V 2884 5300 50  0000 C CNN
 F 2 "Inductor_THT:L_Toroid_Vertical_L10.0mm_W5.0mm_P5.08mm_Diagonal" H 2750 5300 50  0001 C CNN
 F 3 "~" H 2750 5300 50  0001 C CNN
@@
 P 3000 5550
 F 0 "C13" H 3115 5596 50  0000 L CNN
-F 1 "1n" H 3115 5505 50  0000 L CNN
+F 1 "680p" H 3115 5505 50  0000 L CNN
 F 2 "Capacitor_THT:C_Disc_D3.0mm_W1.6mm_P2.50mm" H 3038 5400 50  0001 C CNN
 F 3 "~" H 3000 5550 50  0001 C CNN
@@
 P 3250 5300
 F 0 "L11" V 3475 5300 50  0000 C CNN
-F 1 "1460n" V 3384 5300 50  0000 C CNN
+F 1 "1330n" V 3384 5300 50  0000 C CNN
 F 2 "Inductor_THT:L_Toroid_Vertical_L10.0mm_W5.0mm_P5.08mm_Diagonal" H 3250 5300 50  0001 C CNN
 F 3 "~" H 3250 5300 50  0001 C CNN
@@
 P 3500 5550
 F 0 "C17" H 3615 5596 50  0000 L CNN
-F 1 "680p" H 3615 5505 50  0000 L CNN
+F 1 "330p" H 3615 5505 50  0000 L CNN
 F 2 "Capacitor_THT:C_Disc_D3.0mm_W2.0mm_P2.50mm" H 3538 5400 50  0001 C CNN
 F 3 "~" H 3500 5550 50  0001 C CNN
@@
 P 2250 7100
 F 0 "L4" V 2475 7100 50  0000 C CNN
-F 1 "2520n" V 2384 7100 50  0000 C CNN
+F 1 "2050n" V 2384 7100 50  0000 C CNN
 F 2 "Inductor_THT:L_Toroid_Vertical_L10.0mm_W5.0mm_P5.08mm_Diagonal" H 2250 7100 50  0001 C CNN
 F 3 "~" H 2250 7100 50  0001 C CNN
@@
 P 2000 7350
 F 0 "C5" H 2115 7396 50  0000 L CNN
-F 1 "1n" H 2115 7305 50  0000 L CNN
+F 1 "470p" H 2115 7305 50  0000 L CNN
 F 2 "Capacitor_THT:C_Disc_D3.0mm_W2.0mm_P2.50mm" H 2038 7200 50  0001 C CNN
 F 3 "~" H 2000 7350 50  0001 C CNN
@@
 P 2500 7350
 F 0 "C9" H 2615 7396 50  0000 L CNN
-F 1 "1.8n" H 2615 7305 50  0000 L CNN
+F 1 "1n" H 2615 7305 50  0000 L CNN
 F 2 "Capacitor_THT:C_Disc_D3.0mm_W2.0mm_P2.50mm" H 2538 7200 50  0001 C CNN
 F 3 "~" H 2500 7350 50  0001 C CNN
@@
 P 2750 7100
 F 0 "L8" V 2975 7100 50  0000 C CNN
-F 1 "2780n" V 2884 7100 50  0000 C CNN
+F 1 "3000n" V 2884 7100 50  0000 C CNN
 F 2 "Inductor_THT:L_Toroid_Vertical_L10.0mm_W5.0mm_P5.08mm_Diagonal" H 2750 7100 50  0001 C CNN
 F 3 "~" H 2750 7100 50  0001 C CNN
@@
 P 3000 7350
 F 0 "C14" H 3115 7396 50  0000 L CNN
-F 1 "1.8n" H 3115 7305 50  0000 L CNN
+F 1 "1n" H 3115 7305 50  0000 L CNN
 F 2 "Capacitor_THT:C_Disc_D3.0mm_W1.6mm_P2.50mm" H 3038 7200 50  0001 C CNN
 F 3 "~" H 3000 7350 50  0001 C CNN
@@
 P 3250 7100
 F 0 "L12" V 3475 7100 50  0000 C CNN
-F 1 "2520n" V 3384 7100 50  0000 C CNN
+F 1 "2050n" V 3384 7100 50  0000 C CNN
 F 2 "Inductor_THT:L_Toroid_Vertical_L10.0mm_W5.0mm_P5.08mm_Diagonal" H 3250 7100 50  0001 C CNN
 F 3 "~" H 3250 7100 50  0001 C CNN
@@
 P 3500 7350
 F 0 "C18" H 3615 7396 50  0000 L CNN
-F 1 "1n" H 3615 7305 50  0000 L CNN
+F 1 "470p" H 3615 7305 50  0000 L CNN
 F 2 "Capacitor_THT:C_Disc_D3.0mm_W2.0mm_P2.50mm" H 3538 7200 50  0001 C CNN
 F 3 "~" H 3500 7350 50  0001 C CNN
@@
 Text Notes 2600 3650 0    50   ~ 0
 LP 20m
-Text Notes 2600 5450 0    50   ~ 0
-LP 40m
+Text Notes 2450 4750 0    50   ~ 0
+LP 60m, 40m
 Text Notes 2600 7250 0    50   ~ 0
 LP 80m

Commit message: Fixed minors.
Parts:
- T1: value 10:10@FT37-43 -> 8+8@FT37-43
Changed lines of the file:
@@
 P 7700 2100
 F 0 "T1" H 7700 2478 50  0000 C CNN
-F 1 "10:10@FT37-43" H 7700 2387 50  0000 C CNN
+F 1 "8+8@FT37-43" H 7700 2387 50  0000 C CNN
 F 2 "Transformer_THT:Transformer_Toroid_Vertical_D10.5mm_Amidon-T37" H 7700 2100 50  0001 C CNN
 F 3 "~" H 7700 2100 50  0001 C CNN

Commit message: backup.
Parts:
- T1: footprint Transformer_THT:Transformer_Toroid_Vertical_D10.5mm_Amidon-T37 -> DM3MAT:Transformer_1P_1S_Toroid_Vertical_D10.5mm_Amidon-T37
Changed lines of the file:
@@
 EESchema Schematic File Version 4
 LIBS:pa-cache
-EELAYER 26 0
+EELAYER 29 0
 EELAYER END
 $Descr A4 11693 8268
@@
 F 0 "T1" H 7700 2478 50  0000 C CNN
 F 1 "8+8@FT37-43" H 7700 2387 50  0000 C CNN
-F 2 "Transformer_THT:Transformer_Toroid_Vertical_D10.5mm_Amidon-T37" H 7700 2100 50  0001 C CNN
+F 2 "DM3MAT:Transformer_1P_1S_Toroid_Vertical_D10.5mm_Amidon-T37" H 7700 2100 50  0001 C CNN
 F 3 "~" H 7700 2100 50  0001 C CNN
 	1    7700 2100

Commit message: Added revision 2 hardware.
Parts:
- removed C26: 100n, Capacitor_THT:C_Disc_D3.0mm_W2.0mm_P2.50mm, symbol Device:C
- removed C28: 100u, Capacitor_THT:CP_Radial_D5.0mm_P2.50mm, symbol Device:CP
- removed J10: TX5V, Connector_PinHeader_2.54mm:PinHeader_1x02_P2.54mm_Vertical, symbol Connector_Generic:Conn_01x02
- removed J12, J8: 12V, Connector_PinHeader_2.54mm:PinHeader_1x02_P2.54mm_Vertical, symbol Connector_Generic:Conn_01x02
- removed J2: 20m, Connector_PinHeader_2.54mm:PinHeader_1x02_P2.54mm_Vertical, symbol Connector_Generic:Conn_01x02
- removed J3: 40m, Connector_PinHeader_2.54mm:PinHeader_1x02_P2.54mm_Vertical, symbol Connector_Generic:Conn_01x02
- removed J4: 80m, Connector_PinHeader_2.54mm:PinHeader_1x02_P2.54mm_Vertical, symbol Connector_Generic:Conn_01x02
- removed J5: Key5V, Connector_PinHeader_2.54mm:PinHeader_1x02_P2.54mm_Vertical, symbol Connector_Generic:Conn_01x02
- removed J9: 10m, Connector_PinHeader_2.54mm:PinHeader_1x02_P2.54mm_Vertical, symbol Connector_Generic:Conn_01x02
- removed K1, K2, K3, K4: FINDER-30.22, Relay_THT:Relay_DPDT_Finder_30.22, symbol Relay:FINDER-30.22
- removed U2: L78L05_TO92, Package_TO_SOT_THT:TO-92_Inline_Wide, symbol Regulator_Linear:L78L05_TO92
- added C26: 220u, Capacitor_THT:CP_Radial_D6.3mm_P2.50mm, symbol Device:CP
- added C28: 100n, Capacitor_THT:C_Disc_D4.3mm_W1.9mm_P5.00mm, symbol Device:C
- added C29, C30: 100n, Capacitor_THT:C_Disc_D3.0mm_W2.0mm_P2.50mm, symbol Device:C
- added H1, H2, H3, H4: GND, MountingHole:MountingHole_3.2mm_M3_Pad_Via, symbol Mechanical:MountingHole_Pad
- added J2: FromRX, Connector_PinSocket_2.54mm:PinSocket_1x08_P2.54mm_Vertical, symbol Connector_Generic:Conn_01x08
- added J3: Barrel_Jack_Switch, Connector_BarrelJack:BarrelJack_Wuerth_6941xx301002, symbol Connector:Barrel_Jack_Switch
- added K1, K2, K3, K4: G6S-2, Relay_THT:Relay_DPDT_Omron_G6S-2, symbol Relay:G6S-2
- added L13: 100u, Inductor_THT:L_Axial_L7.0mm_D3.3mm_P10.16mm_Horizontal_Fastron_MICC, symbol Device:L_Core_Ferrite
- C1, C10, C19, C27: footprint Capacitor_THT:C_Rect_L9.0mm_W2.5mm_P7.50mm_MKT -> Capacitor_THT:C_Disc_D3.0mm_W2.0mm_P2.50mm
- C21: footprint Capacitor_THT:C_Disc_D3.0mm_W1.6mm_P2.50mm -> Capacitor_THT:C_Disc_D4.3mm_W1.9mm_P5.00mm
- C24: footprint Capacitor_THT:C_Disc_D3.0mm_W2.0mm_P2.50mm -> Capacitor_THT:C_Disc_D4.7mm_W2.5mm_P5.00mm
- C25: footprint Capacitor_THT:C_Disc_D3.0mm_W2.0mm_P2.50mm -> Capacitor_THT:C_Disc_D4.3mm_W1.9mm_P5.00mm
- J1: footprint Connector_Coaxial:BNC_horizontal -> Connector_Coaxial:BNC_Amphenol_B6252HB-NPP3G-50_Horizontal
- J11: value 12V-PA -> RXSupply; footprint Connector_PinHeader_2.54mm:PinHeader_1x02_P2.54mm_Vertical -> Connector_PinSocket_2.54mm:PinSocket_1x02_P2.54mm_Vertical
- J6, J7: footprint Connector_PinHeader_2.54mm:PinHeader_1x02_P2.54mm_Vertical -> Connector_PinSocket_2.54mm:PinSocket_1x02_P2.54mm_Vertical
- L1, L3, L5, L7: footprint Inductor_THT:L_Toroid_Vertical_L10.0mm_W5.0mm_P5.08mm_Diagonal -> DM3MAT:L_Toroid_Vertical_L10.0mm_W5.0mm_P5.08mm_Diagonal_Rev
- L10, L11, L12, L2, L4, L6, L8, L9: footprint Inductor_THT:L_Toroid_Vertical_L10.0mm_W5.0mm_P5.08mm_Diagonal -> DM3MAT:L_Toroid_Vertical_L10.0mm_W5.0mm_P5.08mm_Diagonal
- Q5: footprint Package_TO_SOT_THT:TO-126-3_Vertical -> Package_TO_SOT_THT:TO-126-3_Horizontal_TabDown
- R10: footprint Resistor_THT:R_Axial_DIN0207_L6.3mm_D2.5mm_P15.24mm_Horizontal -> Resistor_THT:R_Axial_DIN0207_L6.3mm_D2.5mm_P2.54mm_Vertical
- R12: footprint Resistor_THT:R_Axial_DIN0207_L6.3mm_D2.5mm_P10.16mm_Horizontal -> Resistor_THT:R_Axial_DIN0207_L6.3mm_D2.5mm_P7.62mm_Horizontal
- R14: footprint Resistor_THT:R_Axial_DIN0204_L3.6mm_D1.6mm_P2.54mm_Vertical -> Resistor_THT:R_Axial_DIN0204_L3.6mm_D1.6mm_P5.08mm_Horizontal
Connections:
- wire segments 270 -> 278
- no-connect marks 0 -> 1
Other:
- moved on the sheet: D4, J11, R13, U1E
