File: hardware/mech/mech.kicad_pcb (KiCad board)
At the start: 2 copper layers, 105 x 54 mm, 8 parts

Commit message: Started german manual.
Other:
- board text added: "Drillplan for front panel using Fisher chassis."
Changed lines of the file:
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@@
-(kicad_pcb (version 20171130) (host pcbnew 5.1.6-c6e7f7d~86~ubuntu18.04.1)
+(kicad_pcb (version 20171130) (host pcbnew 5.1.5+dfsg1-2build2)
   (general
     (thickness 1.6)
-    (drawings 72)
+    (drawings 73)
     (tracks 0)
     (zones 0)
@@
       (net 1 GND))
   )
+  (gr_text "Drillplan for front panel using Fisher chassis." (at 133.01 36.5) (layer Cmts.User)
+    (effects (font (size 1 1) (thickness 0.15)))
+  )
   (gr_text "4 x M2.5" (at 148.5 54.5) (layer Cmts.User)
